File: BEESP12.brd (EAGLE design)
At the start: 31.7 x 24.4 mm, 11 parts, among them IC1 ESP12

Commit message: Initial project import
Parts:
- S1, S2: device freetronics-master-v1:TACTILE_SWITCH_SMD_2PIN_TINY -> freetronics-jon:TACTILE_SWITCH_SMD_2PIN_TINY
Other:
- board text added: "(c)2015 Superhouse Automation"
- board text added: "superhouse.tv/beesp12"
- board text removed: "(c)2015 Freetronics Pty Ltd Released under the TAPR Open Hardware License tapr.org/OHL"
- board text removed: "Freetronics"
- board text removed: "tron.cc/beesp12"
Changed lines of the file:
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@@
 <layer number="25" name="tNames" color="15" fill="1" visible="no" active="yes"/>
 <layer number="26" name="bNames" color="7" fill="1" visible="no" active="yes"/>
-<layer number="27" name="tValues" color="7" fill="1" visible="no" active="yes"/>
+<layer number="27" name="tValues" color="7" fill="1" visible="yes" active="yes"/>
 <layer number="28" name="bValues" color="7" fill="1" visible="no" active="yes"/>
 <layer number="29" name="tStop" color="7" fill="3" visible="no" active="yes"/>
@@
 <layer number="42" name="bRestrict" color="1" fill="10" visible="no" active="yes"/>
 <layer number="43" name="vRestrict" color="2" fill="10" visible="no" active="yes"/>
-<layer number="44" name="Drills" color="7" fill="1" visible="no" active="yes"/>
+<layer number="44" name="Drills" color="7" fill="1" visible="yes" active="yes"/>
 <layer number="45" name="Holes" color="7" fill="1" visible="yes" active="yes"/>
 <layer number="46" name="Milling" color="3" fill="1" visible="no" active="yes"/>
@@
 <wire x1="6.2738" y1="24.384" x2="0" y2="18.0594" width="0" layer="20"/>
 <wire x1="0" y1="18.0594" x2="0" y2="6.3246" width="0" layer="20"/>
-<text x="3.6584" y="17.7768" size="1.27" layer="22" font="vector" ratio="15" rot="MR270">Freetronics</text>
 <text x="31.1654" y="14.1192" size="0.8636" layer="21" font="vector" ratio="15" rot="R90">v1.0</text>
 <text x="9.906" y="2.386" size="0.8128" layer="21" ratio="15">RX</text>
@@
 <text x="5.334" y="2.386" size="0.8128" layer="21" ratio="15">3V3</text>
 <text x="13.662" y="2.386" size="0.8128" layer="21" ratio="15">RST</text>
-<text x="26.27" y="5.2432" size="1.016" layer="21" font="vector" ratio="15" rot="R90">tron.cc/beesp12</text>
-<wire x1="1.982" y1="17.472" x2="1.982" y2="6.55" width="0.254" layer="22"/>
-<wire x1="1.982" y1="6.55" x2="2.998" y2="5.534" width="0.254" layer="22" curve="90"/>
-<wire x1="2.998" y1="5.534" x2="4.014" y2="6.55" width="0.254" layer="22" curve="90"/>
-<wire x1="4.014" y1="6.55" x2="4.014" y2="17.472" width="0.254" layer="22"/>
-<wire x1="4.014" y1="17.472" x2="2.998" y2="18.488" width="0.254" layer="22" curve="90"/>
-<wire x1="2.998" y1="18.488" x2="1.982" y2="17.472" width="0.254" layer="22" curve="90"/>
+<text x="26.27" y="2.9572" size="1.016" layer="21" font="vector" ratio="15" rot="R90">superhouse.tv/beesp12</text>
 <text x="3.0734" y="10.1092" size="0.9144" layer="21" font="vector" ratio="15" rot="R90">ESP-12</text>
 <text x="31.0134" y="20.9772" size="1.27" layer="21" font="vector" ratio="15" rot="R90" align="bottom-center">RESET</text>
@@
 <wire x1="7.5" y1="2.2" x2="7.5" y2="0.2" width="0.254" layer="21"/>
 <wire x1="9.5" y1="2.2" x2="9.5" y2="0.2" width="0.254" layer="21"/>
-<text x="30.1752" y="9.6106" size="1.016" layer="22" font="vector" ratio="15" rot="MR0">(c)2015 Freetronics Pty Ltd
-Released under the TAPR Open
-Hardware License tapr.org/OHL</text>
+<text x="31.1912" y="2.2446" size="1.016" layer="22" font="vector" ratio="15" rot="MR0">(c)2015 Superhouse Automation</text>
 <text x="29.4132" y="18.4366" size="1.4224" layer="22" font="vector" ratio="15" rot="MR0">ESP-12 WiFi Breakout</text>
-<text x="30.1752" y="14.1986" size="1.4224" layer="22" font="vector" ratio="15" rot="MR0">tron.cc/beesp12</text>
-<text x="25.3492" y="3.3086" size="1.4224" layer="22" font="vector" ratio="15" rot="MR0">SKU: BEESP12</text>
+<text x="30.6832" y="3.7846" size="1.4224" layer="22" font="vector" ratio="15" rot="MR0">superhouse.tv/beesp12</text>
+<text x="3.5494" y="19.7612" size="1.4224" layer="22" font="vector" ratio="15" rot="MR270">SKU: BEESP12</text>
 <text x="31.0134" y="0.4572" size="1.27" layer="21" font="vector" ratio="15" rot="R90">PROGRAM</text>
 <wire x1="13.5" y1="2.2" x2="11.5" y2="2.2" width="0.254" layer="21"/>
@@
 <wire x1="21.5" y1="24.2" x2="19.5" y2="24.2" width="0.254" layer="21"/>
 <wire x1="21.5" y1="22.2" x2="19.5" y2="22.2" width="0.254" layer="21"/>
+<wire x1="21.844" y1="9.906" x2="23.368" y2="6.604" width="0.4064" layer="22" curve="-309.2564"/>
+<wire x1="21.844" y1="9.906" x2="24.13" y2="9.144" width="0.4064" layer="22" curve="163.361194"/>
+<wire x1="24.13" y1="9.144" x2="23.622" y2="12.192" width="0.4064" layer="22"/>
+<wire x1="24.638" y1="7.874" x2="28.448" y2="7.874" width="0.4064" layer="22"/>
+<wire x1="28.448" y1="7.874" x2="27.686" y2="11.43" width="0.4064" layer="22"/>
+<wire x1="23.114" y1="11.176" x2="28.448" y2="11.176" width="0.254" layer="22"/>
+<wire x1="28.448" y1="11.176" x2="25.654" y2="12.954" width="0.254" layer="22"/>
+<wire x1="25.654" y1="12.954" x2="23.114" y2="11.176" width="0.254" layer="22"/>
+<wire x1="27.94" y1="11.43" x2="27.686" y2="11.43" width="0.254" layer="22"/>
+<wire x1="27.686" y1="11.43" x2="23.876" y2="11.43" width="0.254" layer="22"/>
+<wire x1="23.876" y1="11.43" x2="25.654" y2="12.7" width="0.254" layer="22"/>
+<wire x1="25.654" y1="12.7" x2="27.686" y2="11.43" width="0.254" layer="22"/>
+<wire x1="24.384" y1="11.684" x2="27.178" y2="11.684" width="0.4064" layer="22"/>
+<wire x1="27.178" y1="11.684" x2="25.654" y2="12.446" width="0.4064" layer="22"/>
+<wire x1="25.654" y1="12.446" x2="24.892" y2="11.938" width="0.4064" layer="22"/>
+<wire x1="24.892" y1="11.938" x2="26.162" y2="11.938" width="0.4064" layer="22"/>
+<wire x1="26.162" y1="11.938" x2="25.654" y2="12.192" width="0.4064" layer="22"/>
 </plain>
 <attributes>
@@
 <element name="IC1" library="freetronics-jon" package="ESP12" value="ESP12" x="13.208" y="12.192" smashed="yes">
 <attribute name="NAME" x="7.858" y="7.5" size="1.016" layer="25"/>
-<attribute name="VALUE" x="11.16" y="7.294" size="1.016" layer="27"/>
-</element>
-<element name="S1" library="freetronics-master-v1" package="TACTILE_SWITCH_SMD_2PIN_TINY" value="RESET" x="27.94" y="20.828" smashed="yes" rot="R90"/>
+<attribute name="VALUE" x="11.414" y="12.374" size="0.8128" layer="27"/>
+</element>
+<element name="S1" library="freetronics-jon" package="TACTILE_SWITCH_SMD_2PIN_TINY" value="RESET" x="27.94" y="20.828" smashed="yes" rot="R90"/>
 <element name="C1" library="freetronics-master-v1.1" package="0603" value="100nF" x="27.94" y="16.764" smashed="yes">
 <attribute name="NAME" x="29.337" y="16.256" size="1.016" layer="25" font="vector"/>
-<attribute name="VALUE" x="29.21" y="17.3228" size="1.016" layer="27" font="vector"/>
+<attribute name="VALUE" x="29.21" y="16.3068" size="0.8128" layer="27" font="vector"/>
 </element>
 <element name="R1" library="freetronics-master-v1.1" package="0603" value="22K" x="27.94" y="14.986" smashed="yes">
 <attribute name="NAME" x="29.337" y="14.478" size="1.016" layer="25" font="vector"/>
-<attribute name="VALUE" x="29.21" y="14.5288" size="1.016" layer="27" font="vector"/>
-</element>
-<element name="S2" library="freetronics-master-v1" package="TACTILE_SWITCH_SMD_2PIN_TINY" value="PROGRAM" x="27.94" y="3.556" smashed="yes" rot="R270"/>
+<attribute name="VALUE" x="29.21" y="14.5288" size="0.8128" layer="27" font="vector"/>
+</element>
+<element name="S2" library="freetronics-jon" package="TACTILE_SWITCH_SMD_2PIN_TINY" value="PROGRAM" x="27.94" y="3.556" smashed="yes" rot="R270"/>
 <element name="R2" library="freetronics-master-v1.1" package="0603" value="22k" x="27.94" y="7.62" smashed="yes">
 <attribute name="NAME" x="29.337" y="7.112" size="1.016" layer="25" font="vector"/>
-<attribute name="VALUE" x="29.21" y="7.1628" size="1.016" layer="27" font="vector"/>
+<attribute name="VALUE" x="29.21" y="7.1628" size="0.8128" layer="27" font="vector"/>
 </element>
 <element name="R4" library="freetronics-master-v1.1" package="0603" value="22K" x="27.94" y="11.176" smashed="yes">
 <attribute name="NAME" x="29.337" y="10.668" size="1.016" layer="25" font="vector"/>
-<attribute name="VALUE" x="26.924" y="10.2108" size="0.4064" layer="27" font="vector"/>
+<attribute name="VALUE" x="29.21" y="10.9728" size="0.8128" layer="27" font="vector"/>
 </element>
 <element name="R3" library="freetronics-master-v1.1" package="0603" value="22K" x="27.94" y="13.208" smashed="yes" rot="R180">
 <attribute name="NAME" x="29.337" y="12.7" size="1.016" layer="25" font="vector"/>
-<attribute name="VALUE" x="28.956" y="14.1732" size="0.4064" layer="27" font="vector" rot="R180"/>
+<attribute name="VALUE" x="29.21" y="13.0048" size="0.8128" layer="27" font="vector"/>
 </element>
 <element name="R5" library="freetronics-master-v1.1" package="0603" value="22K" x="27.94" y="9.398" smashed="yes">
 <attribute name="NAME" x="29.337" y="8.89" size="1.016" layer="25" font="vector"/>
-<attribute name="VALUE" x="26.924" y="8.4328" size="0.4064" layer="27" font="vector"/>
+<attribute name="VALUE" x="29.21" y="8.9408" size="0.8128" layer="27" font="vector"/>
 </element>
 </elements>
@@
 </board>
 </drawing>
-<compatibility>
-<note version="6.3" minversion="6.2.2" severity="warning">
-Since Version 6.2.2 text objects can contain more than one line,
-which will not be processed correctly with this version.
-</note>
-</compatibility>
 </eagle>
