File: BEESP12.sch (EAGLE design)
At the start: 11 parts, among them IC1 ESP12

Commit message: Initial project import
Parts:
- S1, S2: device freetronics-master-v1:TAC_SWITCH_2PIN -> freetronics-jon:TAC_SWITCH_2PIN
Other:
- note added: "superhouse.tv/beesp12"
- note removed: "tron.cc/beesp12"
Changed lines of the file:
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@@
 <part name="SJ2" library="freetronics-jon" deviceset="SJC" device="N" value="RESET LINK"/>
 <part name="IC1" library="freetronics-jon" deviceset="ESP12" device=""/>
-<part name="S1" library="freetronics-master-v1" deviceset="TAC_SWITCH_2PIN" device="" value="RESET"/>
+<part name="S1" library="freetronics-jon" deviceset="TAC_SWITCH_2PIN" device="" value="RESET"/>
 <part name="GND1" library="supply1" deviceset="GND" device=""/>
 <part name="C1" library="freetronics-master-v1.1" deviceset="CAP" device="0603" value="100nF"/>
@@
 <part name="GND3" library="supply1" deviceset="GND" device=""/>
 <part name="GND4" library="supply1" deviceset="GND" device=""/>
-<part name="S2" library="freetronics-master-v1" deviceset="TAC_SWITCH_2PIN" device="" value="PROGRAM"/>
+<part name="S2" library="freetronics-jon" deviceset="TAC_SWITCH_2PIN" device="" value="PROGRAM"/>
 <part name="GND5" library="supply1" deviceset="GND" device=""/>
 <part name="R2" library="freetronics-master-v1.1" deviceset="RESISTOR" device="0603" value="22k"/>
@@
 <text x="7.62" y="12.7" size="2.794" layer="94">ESP-12 / XBee WiFi Breakout</text>
 <text x="81.28" y="6.858" size="1.778" layer="94">V1.0 (2015-04-22)</text>
-<text x="35.306" y="6.858" size="1.778" layer="94">tron.cc/beesp12</text>
+<text x="35.306" y="6.858" size="1.778" layer="94">superhouse.tv/beesp12</text>
 <frame x1="0" y1="0" x2="248.92" y2="185.42" columns="8" rows="5" layer="94"/>
 <frame x1="5.08" y1="5.08" x2="109.22" y2="17.78" columns="0" rows="0" layer="94" border-left="no" border-top="no" border-right="no" border-bottom="no"/>
